Commit message: Adding rsdf and update the robot model.

File: sawyer_description/urdf/sawyer.urdf (robot description, URDF)
Before this commit: robot sawyer, 36 links, 35 joints
Links:
- removed link head_camera_optical
- removed link right_connector_plate_base
- removed link right_connector_plate_mount
- removed link right_electric_gripper_base
- removed link right_gripper_base
- removed link right_gripper_l_finger
- removed link right_gripper_l_finger_tip
- removed link right_gripper_r_finger
- removed link right_gripper_r_finger_tip
- removed link right_gripper_tip
- removed link right_hand_camera_optical
- removed link world
- link right_arm_itb: mass None -> 0.0001
- link right_hand: mass 0.01 -> 1.0E-08
- link right_l1_2: mass None -> 1.0E-08
- link right_l2_2: mass None -> 1.0E-08
- link right_l4_2: mass None -> 1.0E-08
- link right_torso_itb: mass None -> 0.0001
- link screen: mass None -> 0.0001
- link torso: mass None -> 0.0001
Joints:
- removed joint fixed
- removed joint head_camera_optical_joint
- removed joint right_connector_plate_base_joint
- removed joint right_connector_plate_mount_joint
- removed joint right_electric_gripper_base_joint
- removed joint right_gripper_base_joint
- removed joint right_gripper_l_finger_joint
- removed joint right_gripper_l_finger_tip_joint
- removed joint right_gripper_r_finger_joint
- removed joint right_gripper_r_finger_tip_joint
- removed joint right_gripper_tip_joint
- removed joint right_hand_camera_optical_joint
- joint right_j6: limit lower=-3.14 upper=3.14 effort=9.0 velocity=4.545 -> lower=-4.7124 upper=4.7124 effort=9.0 velocity=4.545
